File: extras/kicad/Baofeng-PTT/Baofeng-PTT.sch (KiCad schematic (older format))
At the start: 18 parts, among them J1 AI, J2 AO, J3 Conn_01x02_Male, J4 PTT, J5 Conn_01x02_Male, J6 Conn_01x02_Male, J7 Conn_01x02_Male, J8 Baofeng, U1 ULN2003

Commit message: Cleanup kikad
Parts:
- removed C1, C2: C1uf, Capacitor_THT:C_Disc_D3.0mm_W1.6mm_P2.50mm, symbol Device:C
- removed D1: DIODE, Diode_THT:D_A-405_P7.62mm_Horizontal, symbol pspice:DIODE
- removed J3, J5, J6, J7: Conn_01x02_Male, Connector_PinHeader_2.54mm:PinHeader_1x02_P2.54mm_Vertical, symbol Connector:Conn_01x02_Male
- removed R1, R6: R1.5k, Resistor_THT:R_Axial_DIN0204_L3.6mm_D1.6mm_P2.54mm_Vertical, symbol Device:R
- removed R2, R5: R15k, Resistor_THT:R_Axial_DIN0204_L3.6mm_D1.6mm_P2.54mm_Vertical, symbol Device:R
- removed R3, R4: R300, Resistor_THT:R_Axial_DIN0204_L3.6mm_D1.6mm_P2.54mm_Vertical, symbol Device:R
- added FB1, FB2, FB3, FB4: Ferrite_Bead, Connector_PinHeader_2.54mm:PinHeader_1x02_P2.54mm_Vertical, symbol Device:Ferrite_Bead
- added R0: R0, Resistor_THT:R_Axial_DIN0207_L6.3mm_D2.5mm_P7.62mm_Horizontal, symbol pspice:R
Connections:
- wire segments 22 -> 12
Other:
- note added: "(Optional) Ferrite beads FB0-FB4\nusing for filtering audio\n\n"
- note removed: "Tor coil"
- moved on the sheet: J4, J8

Commit message: Cleanup Kikad project
Parts:
- removed R0: R0, Resistor_THT:R_Axial_DIN0207_L6.3mm_D2.5mm_P7.62mm_Horizontal, symbol pspice:R
- added J3, J5: Conn_01x15, Connector_PinSocket_2.54mm:PinSocket_1x15_P2.54mm_Vertical, symbol Connector_Generic:Conn_01x15
Connections:
- net GND: now also J5.2 (Pin_2)
- net at U1.1 (I1): now also J4.1 (Pin_1)
- new net DATA: J5.8 (Pin_8)
Changed lines of the file:
@@
 Wire Wire Line
 	1100 2950 1100 2750
-Text GLabel 1000 1000 0    50   Input ~ 0
-PIN
-Text GLabel 1000 1100 0    50   Input ~ 0
-GND
 $Comp
 L Connector:AudioJack3 J1
@@
 F 3 "~" H 1000 3700 50  0001 C CNN
 	1    1000 3700
-	1    0    0    -1
-$EndComp
-$Comp
-L Connector:Conn_01x02_Male J4
-U 1 1 5EFD44E9
-P 1000 1000
-F 0 "J4" H 1250 950 50  0000 C CNN
-F 1 "PTT" H 900 1150 50  0000 C CNN
-F 2 "Connector_PinHeader_2.54mm:PinHeader_1x02_P2.54mm_Vertical" H 1000 1000 50  0001 C CNN
-F 3 "~" H 1000 1000 50  0001 C CNN
-	1    1000 1000
 	1    0    0    -1
 $EndComp
@@
 Wire Wire Line
 	1800 2950 1800 2800
+Text Notes 1450 3350 0    50   ~ 0
+(Optional) Ferrite beads FB0-FB4\nusing for filtering audio\n\n
 $Comp
-L pspice:R R0
-U 1 1 60F7F084
-P 1450 1000
-F 0 "R0" V 1245 1000 50  0000 C CNN
-F 1 "R0" V 1336 1000 50  0000 C CNN
-F 2 "Resistor_THT:R_Axial_DIN0207_L6.3mm_D2.5mm_P7.62mm_Horizontal" H 1450 1000 50  0001 C CNN
-F 3 "~" H 1450 1000 50  0001 C CNN
-	1    1450 1000
+L Connector_Generic:Conn_01x15 J5
+U 1 1 60F3A410
+P 4450 1450
+F 0 "J5" H 4530 1492 50  0000 L CNN
+F 1 "Conn_01x15" H 4530 1401 50  0000 L CNN
+F 2 "Connector_PinSocket_2.54mm:PinSocket_1x15_P2.54mm_Vertical" H 4530 1355 50  0001 L CNN
+F 3 "~" H 4450 1450 50  0001 C CNN
+	1    4450 1450
+	1    0    0    -1
+$EndComp
+$Comp
+L Connector_Generic:Conn_01x15 J3
+U 1 1 60F41DC4
+P 3400 1450
+F 0 "J3" H 3480 1492 50  0000 L CNN
+F 1 "Conn_01x15" H 3480 1401 50  0000 L CNN
+F 2 "Connector_PinSocket_2.54mm:PinSocket_1x15_P2.54mm_Vertical" H 3400 1450 50  0001 C CNN
+F 3 "~" H 3400 1450 50  0001 C CNN
+	1    3400 1450
+	1    0    0    -1
+$EndComp
+$Comp
+L power:GND #PWR0106
+U 1 1 60F445B7
+P 4250 850
+F 0 "#PWR0106" H 4250 600 50  0001 C CNN
+F 1 "GND" H 4255 677 50  0000 C CNN
+F 2 "" H 4250 850 50  0001 C CNN
+F 3 "" H 4250 850 50  0001 C CNN
+	1    4250 850
 	0    1    1    0
 $EndComp
-Text Notes 1450 3350 0    50   ~ 0
-(Optional) Ferrite beads FB0-FB4\nusing for filtering audio\n\n
+Wire Wire Line
+	1200 1000 1700 1000
+$Comp
+L Connector:Conn_01x02_Male J4
+U 1 1 5EFD44E9
+P 1000 1000
+F 0 "J4" H 1250 950 50  0000 C CNN
+F 1 "PTT" H 900 1150 50  0000 C CNN
+F 2 "Connector_PinHeader_2.54mm:PinHeader_1x02_P2.54mm_Vertical" H 1000 1000 50  0001 C CNN
+F 3 "~" H 1000 1000 50  0001 C CNN
+	1    1000 1000
+	1    0    0    -1
+$EndComp
+Text GLabel 1000 1100 0    50   Input ~ 0
+GND
+Text GLabel 1000 1000 0    50   Input ~ 0
+DATA
+Text GLabel 3750 1050 0    50   Input ~ 0
+DATA
+Wire Wire Line
+	4150 1450 4250 1450
+Wire Wire Line
+	4150 1050 4150 1450
+Wire Wire Line
+	3750 1050 4150 1050
 $EndSCHEMATC
